Commit message: Adjust the initial posture to open

File: urdf/rohand_left.urdf (robot description, URDF)
Before this commit: robot rohand_left, 26 links, 25 joints
Links:
- link base_link: mass 0.0367658161456593 -> 0.0278705630237158
- link if_connecting_link: mass 0.000166924672312448 -> 0.000166924761349137
- link if_distal_link: mass 0.00375858037616174 -> 0.0037519230425627
- link if_proximal_link: mass 0.0020519557292877 -> 0.00205188510009486
- link if_slider_abpart_link: mass 0.000320776967954908 -> 0.000302366045011765
- link if_slider_link: mass 0.000366976779244888 -> 0.000366987168246213
- link lf_connecting_link: mass 0.000153781965229355 -> 0.000153788163723339
- link lf_distal_link: mass 0.00243586918410262 -> 0.00242864721731241
- link lf_proximal_link: mass 0.00183703203876047 -> 0.00183698470221302
- link lf_slider_abpart_link: mass 0.000320776967954136 -> 0.000302366045380064
- link lf_slider_link: mass 0.000362008073494643 -> 0.000362014721975395
- link mf_connecting_link: mass 0.000182842940071169 -> 0.000182843644330639
- link mf_distal_link: mass 0.00375852857432825 -> 0.00375188378032024
- link mf_proximal_link: mass 0.00248819746655502 -> 0.00248792244521462
- link mf_slider_abpart_link: mass 0.000320776968205779 -> 0.000302366045302568
- link mf_slider_link: mass 0.000366976877786862 -> 0.000366988392309946
- link rf_connecting_link: mass 0.000166924666599283 -> 0.000166924767845685
- link rf_distal_link: mass 0.00375858491630908 -> 0.00375195160064756
- link rf_proximal_link: mass 0.00205195671379772 -> 0.00205190198130636
- link rf_slider_abpart_link: mass 0.000320776968158487 -> 0.000302366044853382
- link rf_slider_link: mass 0.0003669767565826 -> 0.000366987924985724
- link th_connecting_link: mass 0.000246838976516484 -> 0.000266831545079196
- link th_distal_link: mass 0.00464616025042038 -> 0.00460611705629173
- link th_proximal_link: mass 0.00646398971921865 -> 0.0064647269386138
- link th_root_link: mass 0.00195345377003282 -> 0.00195342767450248
- link th_slider_link: mass 0.000954858111723104 -> 0.000449744359058263
Joints:
- joint if_connecting_link: axis 0 -1 0 -> -0.105287313852345 -0.990657832598564 0.086669719353841; origin xyz=-0.11349 0.034413 0.0028462 rpy=3.0548 -0.0091764 -0.10508 -> xyz=-0.113855295097668 0.031177323718743 0.0069690029233957 rpy=0 0 0
- joint if_distal_link: axis 0 1 0 -> -0.105287313852381 -0.990657832598558 0.0866697193538612; origin xyz=-0.030939 0.00036803 0.010438 rpy=3.1416 0 0 -> xyz=-0.032501413592246 0.00312131258134389 -0.000360511482104104 rpy=0 0 0
- joint if_proximal_link: axis 0 -1 0 -> -0.10529 -0.99066 0.08667; origin xyz=-0.10628 0.036856 -0.0014156 rpy=3.0548 -0.0091764 -0.10508 -> xyz=-0.10701 0.030104 0.0030149 rpy=0 0 0
- joint if_slider_abpart_link: axis 0 1 0 -> -0.105287313852347 -0.990657832598563 0.086669719353844; origin xyz=-0.026698 0.0028818 -0.00025213 rpy=-0.087268 -0.0045707 -0.00023228 -> xyz=-0.0265536336160361 0.00278918570178431 -0.000122523139613851 rpy=0 0 0
- joint if_slider_link: axis 1 0 0 -> 0.9945 -0.10466 0.0046058; limit lower=-0.003 upper=0.016 effort=0 velocity=0 -> lower=0 upper=0.019 effort=0 velocity=0; origin xyz=-0.069843 0.025413 -0.0095469 rpy=0.00048469 -0.0046058 -0.10485 -> xyz=-0.072993 0.025746 -0.005722 rpy=0 0 0
- joint lf_connecting_link: axis 0 1 0 -> 0.095895 -0.99161 -0.086708; origin xyz=-0.1124 -0.022708 0.0043038 rpy=0.08682 -0.0083534 0.09568 -> xyz=-0.11213 -0.02563 0.0078874 rpy=0 0 0
- joint lf_distal_link: axis 0 1 0 -> 0.0958951571285379 -0.991607747644689 -0.0867075178419894; origin xyz=-0.026922 -5.0837E-05 -0.010935 rpy=0 0 0 -> xyz=-0.0288204817146589 -0.00288592788924207 -0.00234003718657118 rpy=0 0 0
- joint lf_proximal_link: axis 0 1 0 -> 0.095895 -0.99161 -0.086708; origin xyz=-0.10588 -0.01818 0.00065724 rpy=0.08682 -0.0083534 0.09568 -> xyz=-0.10528 -0.024621 0.0039331 rpy=0 0 0
- joint lf_slider_abpart_link: axis 0 1 0 -> 0.095895 -0.99161 -0.086708; origin xyz=-0.026696 0.0029268 0.00025609 rpy=0.087275 -0.0036108 -0.0016294 -> xyz=-0.026577 -0.0025522 -0.00012295 rpy=0 0 0
- joint lf_slider_link: axis 1 0 0 -> 0.99526 0.097153 0.0047418; limit lower=-0.003 upper=0.016 effort=0 velocity=0 -> lower=0 upper=0.019 effort=0 velocity=0; origin xyz=-0.067893 -0.020252 -0.0086272 rpy=-0.00046288 -0.0047418 0.097308 -> xyz=-0.071046 -0.020554 -0.0048027 rpy=0 0 0
- joint mf_connecting_link: axis 0 1 0 -> -0.0356840742305421 -0.999363106989115 -0.000165031427541866; origin xyz=-0.11719 0.015178 0.0070447 rpy=0.00016503 0 -0.035692 -> xyz=-0.117310785606758 0.0122334776574983 0.0108836352780683 rpy=0 0 0
- joint mf_distal_link: axis 0 1 0 -> -0.0443196166361777 -0.999016857696227 0.00104384863831518; origin xyz=-0.034844 -5.0349E-05 -0.013726 rpy=0.0043984 0.00019026 -0.0075363 -> xyz=-0.0374220342333107 0.00103220768332958 -0.00234460032529154 rpy=0 0 0
- joint mf_proximal_link: axis 0 1 0 -> -0.035684 -0.99936 -0.00016503; origin xyz=-0.11015 0.018475 0.0030758 rpy=0.00016503 0 -0.035692 -> xyz=-0.1104 0.011987 0.0069142 rpy=0 0 0
- joint mf_slider_abpart_link: axis 0 1 0 -> -0.0356840742305532 -0.999363106989114 -0.000165031427574054; origin xyz=-0.026701 0.0028167 0 rpy=0 0.0046708 0.00026078 -> xyz=-0.0266854788763156 0.000875659284168925 -0.000124561682256132 rpy=0 0 0
- joint mf_slider_link: axis 1 0 0 -> 0.99934 -0.035945 0.0046649; limit lower=-0.003 upper=0.016 effort=0 velocity=0 -> lower=0 upper=0.019 effort=0 velocity=0; origin xyz=-0.072667 0.010715 -0.0056801 rpy=0.00016779 -0.0046649 -0.035953 -> xyz=-0.075833 0.010832 -0.0018554 rpy=0 0 0
- joint rf_connecting_link: axis 0 -1 0 -> 0.0341462472620917 -0.999416834394563 0.000157881815450686; origin xyz=-0.11531 -0.0032532 0.0063702 rpy=3.1414 0 0.034153 -> xyz=-0.115216406754209 -0.00651736130223766 0.0102101953824686 rpy=0 0 0
- joint rf_distal_link: axis 0 1 0 -> 0.0255929476651301 -0.999670698313305 0.00186974960873614; origin xyz=-0.030791 0.00036828 0.010696 rpy=-3.1374 0.00011174 0.0076423 -> xyz=-0.0326225722305464 -0.00141340098263117 -0.000388331442014166 rpy=0 0 0
- joint rf_proximal_link: axis 0 -1 0 -> 0.034146 -0.99942 0.00015788; origin xyz=-0.10852 0.00052975 0.0024009 rpy=3.1414 0 0.034153 -> xyz=-0.1083 -0.0062817 0.0062414 rpy=0 0 0
- joint rf_slider_abpart_link: axis 0 1 0 -> 0.0341462472620816 -0.999416834394563 0.000157881815447721; origin xyz=-0.026698 0.0028938 0 rpy=0 0.0047182 -0.00063032 -> xyz=-0.0266834073402385 -0.000932715217024172 -0.00012582741296854 rpy=0 0 0
- joint rf_slider_link: axis 1 0 0 -> 0.99938 0.034777 0.0047127; limit lower=-0.003 upper=0.016 effort=0 velocity=0 -> lower=0 upper=0.019 effort=0 velocity=0; origin xyz=-0.070868 -0.0049857 -0.0063498 rpy=-0.00016399 -0.0047127 0.034784 -> xyz=-0.074034 -0.0050913 -0.0025252 rpy=0 0 0
- joint th_connecting_link: axis 0 0 -1 -> 0.22107 -0.0072128 -0.97523; origin xyz=0.0342999999310514 9.49029098650939E-05 0.00428598656136089 rpy=3.13437975502215 -0.00387873583868189 2.64821280237015 -> xyz=-0.0022878 0.0041796 -0.00054952 rpy=0 0 0
- joint th_distal_link: axis 0 0 -1 -> 0.221066532016197 -0.00721302051295698 -0.9752320548246; origin xyz=-0.0479097598406365 0.0140073523016571 0.000879436248969738 rpy=0 0 0 -> xyz=-0.0444286041423494 0.0237979030872055 -0.00260849049045741 rpy=0 0 0
- joint th_proximal_link: axis 0 0 -1 -> 0.221066352709782 -0.00721284156886669 -0.975232096793423; origin xyz=-0.0281675109233723 0.0206776396558676 -0.010414259606288 rpy=-0.00721290411178693 0.000240878411888333 0.0333895499404722 -> xyz=-0.00361806617521004 0.0208914100398878 -0.0115003932019436 rpy=0 0 0
- joint th_root_link: axis -1 0 0 -> -0.97466 0.033383 -0.22118; origin xyz=-0.02474 0.01826 -0.019216 rpy=0.0075757 -0.22303 -0.034238 -> xyz=-0.045615 0.018979 -0.020109 rpy=0 0 0
- joint th_slider_link: axis -1 0 0 -> -0.74485815899864 0.647835862453437 -0.159671595133163; limit lower=-0.003 upper=0.007 effort=0 velocity=0 -> lower=0 upper=0.01 effort=0 velocity=0; origin xyz=-0.00693753286125505 0.0060015383018569 0.00770000000000735 rpy=3.13340301156162 0 2.64819881385431 -> xyz=-0.0275958189834185 0.0232821329292057 0.00146785262494971 rpy=0 0 0

File: urdf/rohand_right.urdf (robot description, URDF)
Before this commit: robot rohand_right, 26 links, 25 joints
Links:
- link base_link: mass 0.0493249140792959 -> 0.036767125483042
- link if_connecting_link: mass 0.000166926122979652 -> 0.000166925588454653
- link if_distal_link: mass 0.00375868071914677 -> 0.00375207700561759
- link if_proximal_link: mass 0.00205183706838826 -> 0.00205196484818472
- link if_slider_abpart_link: mass 0.000320776973378262 -> 0.000302366083858827
- link if_slider_link: mass 0.000366972973274265 -> 0.00036698643915296
- link lf_connecting_link: mass 0.000153787132130572 -> 0.000153788693422294
- link lf_distal_link: mass 0.00243556509111398 -> 0.0024429507148898
- link lf_proximal_link: mass 0.00183686407359195 -> 0.00183689354838277
- link lf_slider_abpart_link: mass 0.000320776973239087 -> 0.000302366084373525
- link lf_slider_link: mass 0.000362010956124095 -> 0.000362016423224012
- link mf_connecting_link: mass 0.000182841546424983 -> 0.000182843437407094
- link mf_distal_link: mass 0.00375867884267013 -> 0.00375206640497232
- link mf_proximal_link: mass 0.00248843296883051 -> 0.00248820352291794
- link mf_slider_abpart_link: mass 0.000320776973597363 -> 0.000302366084321501
- link mf_slider_link: mass 0.000366973958523744 -> 0.000366986670362037
- link rf_connecting_link: mass 0.000166926124302073 -> 0.000166925583180313
- link rf_distal_link: mass 0.00375873422510174 -> 0.00375142011813841
- link rf_proximal_link: mass 0.00205187294843744 -> 0.00205194161920879
- link rf_slider_abpart_link: mass 0.000320776973678139 -> 0.00030236608370823
- link rf_slider_link: mass 0.000366972980545594 -> 0.000366986915741481
- link th_connecting_link: mass 0.000246838977263949 -> 0.00022981107779302
- link th_distal_link: mass 0.00464616536496131 -> 0.00460659233357567
- link th_proximal_link: mass 0.00646388849033333 -> 0.00646400989225721
- link th_root_link: mass 0.00195350966248874 -> 0.00195342720986922
- link th_slider_link: mass 0.000954853800364086 -> 0.000486787384748644
Joints:
- joint if_connecting_link: axis 0 1 0 -> 0.03586 -0.99559 -0.08667; origin xyz=-0.11562 -0.026397 0.0028757 rpy=0.086779 -0.00311 0.035733 -> xyz=-0.11575 -0.023152 0.006969 rpy=0 0 0
- joint if_distal_link: axis 0 1 0 -> 0.03586 -0.99559 -0.08667; origin xyz=-0.030875 0.00036803 -0.010625 rpy=0 0 0 -> xyz=-0.03264 -0.00084447 -0.00035932 rpy=0 0 0
- joint if_proximal_link: axis 0 1 0 -> 0.03586 -0.99559 -0.08667; origin xyz=-0.10859 -0.029338 -0.0013861 rpy=0.086779 -0.00311 0.035733 -> xyz=-0.10885 -0.022559 0.0030149 rpy=0 0 0
- joint if_slider_abpart_link: axis 0 1 0 -> 0.03586 -0.99559 -0.08667; origin xyz=-0.026698 -0.0028819 -0.0002512 rpy=0.086944 0.0014956 0.00076252 -> xyz=-0.026684 -0.00092834 -0.00012252 rpy=0 0 0
- joint if_slider_link: axis 1 0 0 -> 0.99938 0.034963 0.0046058; limit lower=-0.003 upper=0.016 effort=0 velocity=0 -> lower=0 upper=0.019 effort=0 velocity=0; origin xyz=-0.071447 -0.020467 -0.0095174 rpy=-0.00016113 -0.0046058 0.034971 -> xyz=-0.074613 -0.020587 -0.005722 rpy=0 0 0
- joint lf_connecting_link: axis 0 1 0 -> -0.1649 -0.98249 0.086708; origin xyz=-0.11054 0.030508 0.0043333 rpy=-0.086826 -0.014497 -0.16502 -> xyz=-0.11007 0.033397 0.0078874 rpy=0 0 0
- joint lf_distal_link: axis 0 1 0 -> -0.1649 -0.98249 0.086708; origin xyz=-0.026989 5.0837E-05 -0.010769 rpy=0 0 0 -> xyz=-0.028549 0.0048912 -0.00234 rpy=0 0 0
- joint lf_proximal_link: axis 0 1 0 -> -0.1649 -0.98249 0.086708; origin xyz=-0.10436 0.025536 0.00068678 rpy=-0.086826 -0.014497 -0.16502 -> xyz=-0.1033 0.031912 0.0039331 rpy=0 0 0
- joint lf_slider_abpart_link: axis 0 1 0 -> -0.1649 -0.98249 0.086708; origin xyz=-0.026696 -0.0029267 0.00025708 rpy=-0.087616 -0.0097532 0.0021703 -> xyz=-0.026334 0.0044017 -0.00012295 rpy=0 0 0
- joint lf_slider_link: axis 1 0 0 -> 0.98605 -0.16641 0.0047418; limit lower=-0.003 upper=0.016 effort=0 velocity=0 -> lower=0 upper=0.019 effort=0 velocity=0; origin xyz=-0.066313 0.024951 -0.0085977 rpy=0.00080024 -0.0047418 -0.16719 -> xyz=-0.069437 0.025465 -0.0048027 rpy=0 0 0
- joint mf_connecting_link: axis 0 1 0 -> -0.034181 -0.99942 0.00016502; origin xyz=-0.117961503708004 -0.00695063768300233 0.00707421346498281 rpy=-0.000165024105881287 0 -0.0341875332667273 -> xyz=-0.11788 -0.0040127 0.010884 rpy=0 0 0
- joint mf_distal_link: axis 0 1 0 -> -0.025542 -0.99967 -0.0010432; origin xyz=-0.0348440227740655 5.03497035553302E-05 -0.0137271073982339 rpy=-0.00439882751506536 -0.000117257737364924 0.00753742768873965 -> xyz=-0.037403 0.0015832 -0.0023459 rpy=0 0 0
- joint mf_proximal_link: axis 0 1 0 -> -0.034181 -0.99942 0.00016502; origin xyz=-0.111168350336371 -0.0107315849401363 0.00310533319557881 rpy=-0.000165024105879644 0 -0.0341875332667528 -> xyz=-0.11096 -0.0042498 0.0069142 rpy=0 0 0
- joint mf_slider_abpart_link: axis 0 1 0 -> -0.034181 -0.99942 0.00016502; origin xyz=-0.026701 -0.0028167 0 rpy=-0.00032457 0.0046592 -0.0002623 -> xyz=-0.026681 0.00098972 -0.00012456 rpy=0 0 0
- joint mf_slider_link: axis 1 0 0 -> 0.99941 -0.033919 0.0046649; limit lower=-0.003 upper=0.016 effort=0 velocity=0 -> lower=0 upper=0.019 effort=0 velocity=0; origin xyz=-0.073238 -0.005607 -0.0056506 rpy=0.00015832 -0.0046649 -0.033926 -> xyz=-0.076404 -0.0055105 -0.0018554 rpy=0 0 0
- joint rf_connecting_link: axis 0 1 0 -> -0.10384 -0.99459 -0.00015789; origin xyz=-0.1148 0.011304 0.0063998 rpy=0.00015789 1.6485E-05 -0.10403 -> xyz=-0.11448 0.014546 0.01021 rpy=0 0 0
- joint rf_distal_link: axis 0 1 0 -> -0.09533 -0.99544 -0.0018704; origin xyz=-0.030791 0.00036828 -0.010696 rpy=-0.0042136 -0.0004074 0.0076437 -> xyz=-0.032444 0.0036877 -0.00038717 rpy=0 0 0
- joint rf_proximal_link: axis 0 1 0 -> -0.10384 -0.99459 -0.00015789; origin xyz=-0.10829 0.007056 0.0024304 rpy=0.00015789 1.6485E-05 -0.10403 -> xyz=-0.1076 0.013828 0.0062414 rpy=0 0 0
- joint rf_slider_abpart_link: axis 0 1 0 -> -0.10384 -0.99459 -0.00015789; origin xyz=-0.024396 0.014106 -0.0020413 rpy=-0.087604 -0.0098226 -0.060353 -> xyz=-0.026553 0.0027935 -0.00012583 rpy=0 0 0
- joint rf_slider_link: axis 1 0 0 -> 0.99452 -0.10447 0.0047127; limit lower=-0.003 upper=0.016 effort=0 velocity=0 -> lower=0 upper=0.019 effort=0 velocity=0; origin xyz=-0.070347 0.0099293 -0.0063203 rpy=0.00049505 -0.0047127 -0.10466 -> xyz=-0.073497 0.010248 -0.0025252 rpy=0 0 0
- joint th_connecting_link: axis 0 0 1 -> -0.22103 0.0082401 0.97523; origin xyz=0.0333 -0.00016876 0.0042837 rpy=3.1334 0.0037317 -2.7164 -> xyz=-0.0025078 -0.0040122 -0.00084209 rpy=0 0 0
- joint th_distal_link: axis 0 0 1 -> -0.22103 0.00824 0.97523; origin xyz=-0.048752 -0.010712 0.00087944 rpy=0 0 0 -> xyz=-0.04565 -0.02065 -0.0040713 rpy=0 0 0
- joint th_proximal_link: axis 0 0 1 -> -0.22103 0.0082401 0.97523; origin xyz=-0.028168 -0.020837 -0.010094 rpy=-0.0082402 0.00028649 0.034758 -> xyz=-0.0053995 -0.020575 -0.010038 rpy=0 0 0
- joint th_root_link: axis 1 0 0 -> 0.97461 -0.034751 0.22118; origin xyz=-0.025954 -0.01648 -0.019186 rpy=0.0078865 -0.22303 -0.035641 -> xyz=-0.046829 -0.015748 -0.020109 rpy=0 0 0
- joint th_slider_link: axis 1 0 0 -> -0.78525 -0.59442 -0.17337; limit lower=-0.003 upper=0.007 effort=0 velocity=0 -> lower=0 upper=0.01 effort=0 velocity=0; origin xyz=-0.0082411 -0.0059277 0.0077 rpy=3.1325 0 -2.7163 -> xyz=-0.028823 -0.021311 0 rpy=0 0 0
